Commit message: Se añadieron diferentes carpetas xacro y se editaron sus contenidos "Part No. 1"

File: description/robot.urdf.xacro (robot description, xacro)
@@ -2,6 +2,6 @@
 <robot xmlns:xacro="http://www.ros.org/wiki/xacro"  name="robot">
     <!-- Example link -->
+    <xacro:include filename="properties.xacro"/>
     <xacro:include filename="robot_core.xacro"/>
-        <!-- Example link -->
-    <link name="base_link"></link>
+    <xacro:include filename="inertial_macros.xacro"/>
 </robot>

Commit message: Edición de contenido robot_core.xacro

File: description/robot.urdf.xacro (robot description, xacro)
@@ -4,4 +4,3 @@
     <xacro:include filename="properties.xacro"/>
     <xacro:include filename="robot_core.xacro"/>
-    <xacro:include filename="inertial_macros.xacro"/>
 </robot>

File: description/robot_core.xacro (robot description, xacro)
@@ -34,5 +34,5 @@
         <parent link="base_link"/>
         <child link="left_wheel"/>
-        <origin xyz="0 0.175 0" rpy="-${pi/2} 0 0"/>
+        <origin xyz="0 0.175 0" rpy="-${3.1415926/2} 0 0"/>
         <axis xyz="0 0 1"/>
     </joint>
@@ -58,5 +58,5 @@
         <parent link="base_link"/>
         <child link="right_wheel"/>
-        <origin xyz="0 -0.175 0" rpy="${pi/2} 0 0"/>
+        <origin xyz="0 -0.175 0" rpy="${3.1415926/2} 0 0"/>
         <axis xyz="0 0 -1"/>
     </joint>

Commit message: Se creó el archivo launch_sim.launch.py, se creó el archivo gazebo_control.xacro y se editaron las carpetas robot_core.xacro y robot.urdf.xacro "Parto No. 2"

File: description/robot.urdf.xacro (robot description, xacro)
@@ -4,3 +4,4 @@
     <xacro:include filename="properties.xacro"/>
     <xacro:include filename="robot_core.xacro"/>
+    <xacro:include filename="gazebo_control.xacro"/>
 </robot>

File: description/robot_core.xacro (robot description, xacro)
@@ -29,4 +29,7 @@
             <origin xyz="0.15 0 0.075" rpy="0 0 0"/>
         </xacro:inertial_box>
+        <gazebo reference="chassis">
+            <material>Gazebo/White</material>
+        </gazebo>
     </link>
     <!-- left wheel joint -->
@@ -34,5 +37,5 @@
         <parent link="base_link"/>
         <child link="left_wheel"/>
-        <origin xyz="0 0.175 0" rpy="-${3.1415926/2} 0 0"/>
+        <origin xyz="0 0.175 0" rpy="-${pi/2} 0 0"/>
         <axis xyz="0 0 1"/>
     </joint>
@@ -53,4 +56,7 @@
             <origin xyz="0 0 0" rpy="0 0 0"/>
         </xacro:inertial_cylinder>
+        <gazebo reference="left_wheel">
+            <material>Gazebo/Blue</material>
+        </gazebo>
     </link>
     <!-- right wheel joint -->
@@ -58,5 +64,5 @@
         <parent link="base_link"/>
         <child link="right_wheel"/>
-        <origin xyz="0 -0.175 0" rpy="${3.1415926/2} 0 0"/>
+        <origin xyz="0 -0.175 0" rpy="${pi/2} 0 0"/>
         <axis xyz="0 0 -1"/>
     </joint>
@@ -77,4 +83,7 @@
             <origin xyz="0 0 0" rpy="0 0 0"/>
         </xacro:inertial_cylinder>
+        <gazebo reference="right_wheel">
+            <material>Gazebo/Blue</material>
+        </gazebo>
     </link>
     <!-- caster wheel joint -->
@@ -90,5 +99,5 @@
                 <sphere radius="0.05"/>
             </geometry>
-            <material name="black"/>
+            <material name="red"/>
         </visual>
         <collision>
@@ -100,4 +109,9 @@
             <origin xyz="0 0 0" rpy="0 0 0"/>
         </xacro:inertial_sphere>
+        <gazebo reference="caster_wheel">
+            <material>Gazebo/Black</material>
+            <mu1 value = "0.001" />
+            <mu2 value = "0.001" />
+        </gazebo>
     </link>
 </robot>
